File: IP_Circuit_Schematics/IP_Circuit_Schematics.kicad_sch (KiCad schematic)
At the start: 7 parts, among them J1 p3022 rot sensor, M1 Nema 17

Commit message: Update README and circuit schematic
Parts:
- R1: value 100 ohm -> 220 ohm
Changed lines of the file:
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@@
 			)
 		)
-		(property "Value" "100 ohm"
+		(property "Value" "220 ohm"
 			(at 85.09 91.44 90)
 			(show_name no)
